File: PHASE_B/Uno_Shield_ThermoPro/Uno_Shield_ThermoPro_Template_1/Uno_Shield_ThermoPro.kicad_pcb (KiCad board)
At the start: 2 copper layers, 68.6 x 53.3 mm, 20 parts, among them J1 Power, J2 Digital/PWM, J3 Analog, J4 Digital/PWM, J5 CONN_GYRO, J6 CONN_DISPLAY, J7 CONN_TEMP, SW1 SW_SPST, SW2 SW_SPST, SW3 SW_SPST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

Commit message: update
Routing:
- net +5V: track 186.9 -> 188.1 mm
Other:
- board text added: "Calibrate"
- board text added: "DIsplay"
- board text added: "Light"
- board text added: "Lock"
- board text added: "ON/OFF"
- board text added: "Temp Sensor"
- board text added: "Units"
Changed lines of the file:
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@@
 	(paper "A4")
 	(title_block
-		(date "mar. 31 mars 2015")
+		(title "Uno Shield ThermoPro")
+		(date "2/3/2025")
+		(rev "1.0")
+		(company "Luciano Henriquez")
 	)
 	(layers
@@
 		(tags "Resistor Axial_DIN0207 series Axial Horizontal pin pitch 10.16mm 0.25W = 1/4W length 6.3mm diameter 2.5mm")
 		(property "Reference" "R4"
-			(at 5.01 0.01 360)
+			(at 5.01 0.01 0)
 			(layer "F.SilkS")
 			(effects
@@
 		)
 		(property "Value" "100k"
-			(at 5.08 2.37 360)
+			(at 5.08 2.37 0)
 			(layer "F.Fab")
 			(effects
@@
 		)
 		(fp_text user "${REFERENCE}"
-			(at 5.08 0 360)
+			(at 5.08 0 0)
 			(layer "F.Fab")
 			(effects
@@
 		(tags "Resistor Axial_DIN0207 series Axial Horizontal pin pitch 10.16mm 0.25W = 1/4W length 6.3mm diameter 2.5mm")
 		(property "Reference" "R1"
-			(at 5.12 0.03 360)
+			(at 5.12 0.03 0)
 			(layer "F.SilkS")
 			(effects
@@
 		)
 		(property "Value" "1k"
-			(at 5.08 2.37 360)
+			(at 5.08 2.37 0)
 			(layer "F.Fab")
 			(effects
@@
 		)
 		(fp_text user "${REFERENCE}"
-			(at 5.08 0 360)
+			(at 5.08 0 0)
 			(layer "F.Fab")
 			(effects
@@
 		)
 		(fp_text user "${REFERENCE}"
-			(at 0 3.81 360)
+			(at 0 3.81 0)
 			(layer "F.Fab")
 			(effects
@@
 		(tags "Resistor Axial_DIN0207 series Axial Horizontal pin pitch 10.16mm 0.25W = 1/4W length 6.3mm diameter 2.5mm")
 		(property "Reference" "R5"
-			(at 5.01 -0.01 360)
+			(at 5.01 -0.01 0)
 			(layer "F.SilkS")
 			(effects
@@
 		)
 		(property "Value" "100k"
-			(at 5.08 2.37 360)
+			(at 5.08 2.37 0)
 			(layer "F.Fab")
 			(effects
@@
 		)
 		(fp_text user "${REFERENCE}"
-			(at 5.08 0 360)
+			(at 5.08 0 0)
 			(layer "F.Fab")
 			(effects
@@
 		(tags "Resistor Axial_DIN0207 series Axial Horizontal pin pitch 10.16mm 0.25W = 1/4W length 6.3mm diameter 2.5mm")
 		(property "Reference" "R2"
-			(at 5.01 0.05 360)
+			(at 5.01 0.05 0)
 			(layer "F.SilkS")
 			(effects
@@
 		)
 		(property "Value" "100k"
-			(at 5.08 2.37 360)
+			(at 5.08 2.37 0)
 			(layer "F.Fab")
 			(effects
@@
 		)
 		(fp_text user "${REFERENCE}"
-			(at 5.08 0 360)
+			(at 5.08 0 0)
 			(layer "F.Fab")
 			(effects
@@
 		)
 		(fp_text user "${REFERENCE}"
-			(at 0 8.89 360)
+			(at 0 8.89 0)
 			(layer "F.Fab")
 			(effects
@@
 		(tags "Resistor Axial_DIN0207 series Axial Horizontal pin pitch 10.16mm 0.25W = 1/4W length 6.3mm diameter 2.5mm")
 		(property "Reference" "R6"
-			(at 5.11 -0.07 360)
+			(at 5.11 -0.07 0)
 			(layer "F.SilkS")
 			(effects
@@
 		)
 		(property "Value" "100k"
-			(at 5.08 2.37 360)
+			(at 5.08 2.37 0)
 			(layer "F.Fab")
 			(effects
@@
 		)
 		(fp_text user "${REFERENCE}"
-			(at 5.08 0 360)
+			(at 5.08 0 0)
 			(layer "F.Fab")
 			(effects
@@
 		(tags "Resistor Axial_DIN0207 series Axial Horizontal pin pitch 10.16mm 0.25W = 1/4W length 6.3mm diameter 2.5mm")
 		(property "Reference" "R3"
-			(at 5.13 0.14 360)
+			(at 5.13 0.14 0)
 			(layer "F.SilkS")
 			(effects
@@
 		)
 		(property "Value" "100k"
-			(at 5.08 2.37 360)
+			(at 5.08 2.37 0)
 			(layer "F.Fab")
 			(effects
@@
 		)
 		(fp_text user "${REFERENCE}"
-			(at 5.08 0 360)
+			(at 5.08 0 0)
 			(layer "F.Fab")
 			(effects
@@
 	)
 	(gr_rect
-		(start 101.35 94.3)
-		(end 128.65 66.5)
+		(start 101.35 66.5)
+		(end 128.65 94.3)
 		(stroke
 			(width 0.1)
@@
 		(layer "Edge.Cuts")
 	)
+	(gr_text "Lock"
+		(at 146 94.5 0)
+		(layer "F.SilkS")
+		(effects
+			(font
+				(size 1 1)
+				(thickness 0.15)
+			)
+			(justify left bottom)
+		)
+	)
+	(gr_text "Light"
+		(at 130 95 0)
+		(layer "F.SilkS")
+		(effects
+			(font
+				(size 1 1)
+				(thickness 0.15)
+			)
+			(justify left bottom)
+		)
+	)
+	(gr_text "Units\n"
+		(at 160.5 83.5 0)
+		(layer "F.SilkS")
+		(effects
+			(font
+				(size 1 1)
+				(thickness 0.15)
+			)
+			(justify left bottom)
+		)
+	)
+	(gr_text "DIsplay\n"
+		(at 101.5 68.5 0)
+		(layer "F.SilkS")
+		(effects
+			(font
+				(size 1 1)
+				(thickness 0.15)
+			)
+			(justify left bottom)
+		)
+	)
+	(gr_text "Calibrate"
+		(at 137 73 0)
+		(layer "F.SilkS")
+		(effects
+			(font
+				(size 1 1)
+				(thickness 0.15)
+			)
+			(justify left bottom)
+		)
+	)
+	(gr_text "Temp Sensor\n"
+		(at 103 51.5 0)
+		(layer "F.SilkS")
+		(effects
+			(font
+				(size 1 1)
+				(thickness 0.15)
+			)
+			(justify left bottom)
+		)
+	)
+	(gr_text "ON/OFF"
+		(at 157.5 61.5 0)
+		(layer "F.SilkS")
+		(effects
+			(font
+				(size 1 1)
+				(thickness 0.15)
+			)
+			(justify left bottom)
+		)
+	)
 	(segment
 		(start 147.775 57.8)
@@
 	)
 	(segment
+		(start 125 72.185)
+		(end 122 69.185)
+		(width 0.25)
+		(layer "F.Cu")
+		(net 2)
+	)
+	(segment
 		(start 147.775 59.486701)
 		(end 147.775 57.8)
@@
 	)
 	(segment
-		(start 125 80.373833)
+		(start 122 69.185)
 		(end 125 69.185)
 		(width 0.25)
@@
 	)
 	(segment
+		(start 125 80.373833)
+		(end 125 72.185)
+		(width 0.25)
+		(layer "F.Cu")
+		(net 2)
+	)
+	(segment
 		(start 125 69.185)
 		(end 136.815 69.185)
@@
 	)
 	(segment
+		(start 114.915 69.185)
+		(end 122 69.185)
+		(width 0.25)
+		(layer "F.Cu")
+		(net 2)
+	)
+	(segment
 		(start 146 91.5)
 		(end 152.5 91.5)
@@
 		(width 0.25)
 		(layer "F.Cu")
-		(net 2)
-	)
-	(segment
-		(start 114.915 69.185)
-		(end 125 69.185)
-		(width 0.25)
-		(layer "F.Cu")

Commit message: Uploaded kicad files
Parts:
- added G***: LOGO, LOGO, F.Cu at (107.0, 89.5)
Routing:
- net +5V: track 188.1 -> 187.1 mm
- net /button_units: track 46.6 -> 45.7 mm
- net /button_lock: track 45.7 -> 45.0 mm

Commit message: Uploaded kicad files
Other:
- board text added: "IMU"
- board text added: "TEMP SENSOR"
- board text removed: "Temp Sensor"
Changed lines of the file:
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@@
 		(grid_origin 100 100)
 		(pcbplotparams
-			(layerselection 0x0000030_80000001)
+			(layerselection 0x00010fc_ffffffff)
 			(plot_on_all_layers_selection 0x0000000_00000000)
 			(disableapertmacros no)
@@
 			(outputformat 1)
 			(mirror no)
-			(drillshape 1)
+			(drillshape 0)
 			(scaleselection 1)
-			(outputdirectory "")
+			(outputdirectory "gerber/")
 		)
 	)
@@
 		(at 107 89.5)
 		(property "Reference" "G***"
-			(at 0 0 360)
+			(at 0 0 0)
 			(layer "F.SilkS")
 			(hide yes)
@@
 		)
 		(property "Value" "LOGO"
-			(at 0.75 0 360)
+			(at 0.75 0 0)
 			(layer "F.SilkS")
 			(hide yes)
@@
 		)
 		(property "Footprint" ""
-			(at 0 0 360)
+			(at 0 0 0)
 			(layer "F.Fab")
 			(hide yes)
@@
 		)
 		(property "Datasheet" ""
-			(at 0 0 360)
+			(at 0 0 0)
 			(layer "F.Fab")
 			(hide yes)
@@
 		)
 		(property "Description" ""
-			(at 0 0 360)
+			(at 0 0 0)
 			(layer "F.Fab")
 			(hide yes)
@@
 		)
 	)
-	(gr_text "Temp Sensor\n"
+	(gr_text "TEMP SENSOR\n"
+		(at 125.5 53 0)
+		(layer "F.SilkS")
+		(effects
+			(font
+				(size 1 1)
+				(thickness 0.15)
+			)
+			(justify left bottom)
+		)
+	)
+	(gr_text "IMU\n"
 		(at 103 51.5 0)
 		(layer "F.SilkS")

Commit message: Uploaded kicad files again
Other:
- board text added: "MPU 6050"
- board text added: "OLED TEMU 096"
- board text removed: "DIsplay"
- board text removed: "IMU"
- board text removed: "TEMP SENSOR"
Changed lines of the file:
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@@
 		)
 	)
-	(gr_text "DIsplay\n"
-		(at 101.5 68.5 0)
+	(gr_text "OLED TEMU 096\n"
+		(at 115.5 93 0)
 		(layer "F.SilkS")
 		(effects
@@
 		)
 	)
-	(gr_text "TEMP SENSOR\n"
-		(at 125.5 53 0)
-		(layer "F.SilkS")
-		(effects
-			(font
-				(size 1 1)
-				(thickness 0.15)
-			)
-			(justify left bottom)
-		)
-	)
-	(gr_text "IMU\n"
+	(gr_text "MPU 6050\n"
 		(at 103 51.5 0)
 		(layer "F.SilkS")
