File: PHASE_D/Final Project/final_project_payload/final_project_payload.kicad_sch (KiCad schematic)
At the start: 23 parts, among them J1 Power, J2 Digital/PWM, J3 Analog, J4 Digital/PWM, J5 CONN_PRES, J6 CONN_RTD, J7 CONN_ LIS3DH, U1 GSDA213, U2 AM2302, U3 DEV-13712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

Commit message: test
Other:
- note added: "LUCIANO HENRIQUEZ"
Changed lines of the file:
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@@
+		)
+	)
+	(text "LUCIANO HENRIQUEZ\n"
+		(exclude_from_sim no)
+		(at 187.706 170.434 0)
+		(effects
+			(font
+				(size 1.27 1.27)
+			)
 		)
 	)
